File: persimmon_circle.sch (EAGLE design)
At the start: 34 parts

Commit message: Persimmon circle Rev.Beta1　リファイン
Parts:
- removed LED13: (no value), FaBo-LED:LED-0603
- added 0: (no value), FaBo-LED:APA102_IPIXEL
- LED1: device FaBo-LED:APA102_IPIXEL -> FaBo-LED:LED-0603
- renumbered IC2 to MIC, J1 to I2C, J2 to DEBUG, LED10 to 9, LED11 to 10, LED12 to 11, LED2 to 1, LED3 to 2, LED4 to 3, LED5 to 4, LED6 to 5, LED7 to 6, LED8 to 7, LED9 to 8, USB1 to USB
Connections:
- net N$1 renamed USB_DM
- net N$11 renamed DI1
- net N$12 renamed CI1
- net N$13 renamed DI2
- net N$14 renamed CI2
- net N$15 renamed DI3
- net N$16 renamed CI3
- net N$17 renamed DI4
- net N$18 renamed CI4
- net N$19 renamed DI6
- net N$2 renamed USB_DP
- net N$20 renamed CI6
- net N$21 renamed DI7
- net N$22 renamed CI7
- net N$23 renamed DI8
- net N$24 renamed CI8
- net N$25 renamed DI9
- net N$26 renamed CI9
- net N$27 renamed DI10
- net N$28 renamed CI10
- net N$3 renamed X2
- net N$4 renamed X1
- net N$5 renamed L1
- removed net N$10: 1.CKI, LED1.CKO
- removed net N$6: LED13.ANODE, R3.1
- removed net N$9: 1.SDI, LED1.SDO
- new net CI0: 0.CKO, 1.CKI
- new net DI0: 0.SDO, 1.SDI
- new net LED1: LED1.ANODE, R3.1
- net 5V: now also 0.VCC; no longer LED1.VCC
- net GND: now also 0.GND, LED1.CATHODE; no longer LED1.GND, LED13.CATHODE
- net MOSI: now also 0.SDI; no longer LED1.SDI
- net SCK: now also 0.CKI; no longer LED1.CKI
